Commit message: Latest commit

File: src/v068_description/URDF/denso_vs068A2-AV6-NNN-AA.urdf (robot description, URDF)
Before this commit: robot denso_vs068A2-AV6-NNN-AA, 6 links, 5 joints
Links:
- link link1: mass None -> 3.378
- link link2: mass None -> 7.415
- link link3: mass None -> 1.667
- link link4: mass None -> 1.113
- link link5: mass None -> 0.514
